File: CNChess_KiCad/CNChess_KiCad.kicad_sch (KiCad schematic)
At the start: 32 parts, among them J1 Barrel_Jack, J2 Motor1, J3 Motor2, J4 Servomotor, J5 Fan, SW1 LSW1, SW2 LSW2, SW3 OOSW, U1 ESP32C3, U2 Power_Regulator

Commit message: update elec et TBsem5
Connections:
- net +5V_buck: now reaches J4.2 (Pin_2), U2.5 (OUT+)
- net +5V_buck: now also TP2.1
- net +5V: no longer names the net of U1.14 (5V)
- net +5V: no longer TP2.1
- no-connect marks 15 -> 16
Other:
- moved on the sheet: TP1, TP2, TP3, TP4
Changed lines of the file:
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@@
 	)
 	(no_connect
+		(at 63.5 31.75)
+	)
+	(no_connect
 		(at 99.06 74.93)
 	)
@@
 	(wire
 		(pts
-			(xy 63.5 31.75) (xy 67.31 31.75)
-		)
-		(stroke
-			(width 0)
-			(type default)
-		)
-	)
-	(wire
-		(pts
 			(xy 119.38 44.45) (xy 127 44.45)
 		)
@@
 	(global_label "SW1"
 		(shape input)
-		(at 203.2 72.39 90)
+		(at 203.2 73.66 90)
 		(fields_autoplaced yes)
 		(effects
@@
 		)
 		(property "Intersheetrefs" "${INTERSHEET_REFS}"
-			(at 203.2 65.5344 90)
+			(at 203.2 66.8044 90)
 			(effects
 				(font
@@
 		)
 	)
+	(global_label "+5V_buck"
+		(shape input)
+		(at 127 123.19 90)
+		(fields_autoplaced yes)
+		(effects
+			(font
+				(size 1.27 1.27)
+			)
+			(justify left)
+		)
+		(property "Intersheetrefs" "${INTERSHEET_REFS}"
+			(at 127 110.952 90)
+			(effects
+				(font
+					(size 1.27 1.27)
+				)
+				(justify left)
+				(hide yes)
+			)
+		)
+	)
 	(global_label "SW2"
 		(shape input)
@@
 		)
 	)
+	(global_label "+5V_buck"
+		(shape input)
+		(at 194.31 73.66 90)
+		(fields_autoplaced yes)
+		(effects
+			(font
+				(size 1.27 1.27)
+			)
+			(justify left)
+		)
+		(property "Intersheetrefs" "${INTERSHEET_REFS}"
+			(at 194.31 61.422 90)
+			(effects
+				(font
+					(size 1.27 1.27)
+				)
+				(justify left)
+				(hide yes)
+			)
+		)
+	)
 	(global_label "DIR1"
 		(shape input)
@@
 	(global_label "SW2"
 		(shape input)
-		(at 212.09 72.39 90)
+		(at 212.09 73.66 90)
 		(fields_autoplaced yes)
 		(effects
@@
 		)
 		(property "Intersheetrefs" "${INTERSHEET_REFS}"
-			(at 212.09 65.5344 90)
+			(at 212.09 66.8044 90)
 			(effects
 				(font
@@
 	(symbol
 		(lib_id "Connector:TestPoint")
-		(at 203.2 72.39 180)
+		(at 203.2 73.66 180)
 		(unit 1)
 		(exclude_from_sim no)
@@
 		(dnp no)
 		(property "Reference" "TP3"
-			(at 204.978 81.026 0)
+			(at 204.978 82.296 0)
 			(effects
 				(font
@@
 		)
 		(property "Value" "TPSW1"
-			(at 206.248 78.74 0)
+			(at 206.248 80.01 0)
 			(effects
 				(font
@@
 		)
 		(property "Footprint" "TestPoint:TestPoint_Pad_D1.5mm"
-			(at 198.12 72.39 0)
+			(at 198.12 73.66 0)
 			(effects
 				(font
@@
 		)
 		(property "Datasheet" "~"
-			(at 198.12 72.39 0)
+			(at 198.12 73.66 0)
 			(effects
 				(font
@@
 		)
 		(property "Description" "test point"
-			(at 203.2 72.39 0)
+			(at 203.2 73.66 0)
 			(effects
 				(font
@@
 	(symbol
 		(lib_id "power:+5V")
-		(at 184.15 72.39 0)
+		(at 184.15 73.66 0)
 		(unit 1)
 		(exclude_from_sim no)
@@
 		(fields_autoplaced yes)
 		(property "Reference" "#PWR012"
-			(at 184.15 76.2 0)
+			(at 184.15 77.47 0)
 			(effects
 				(font
@@
 		)
 		(property "Value" "+12V"
-			(at 184.15 67.31 0)
+			(at 184.15 68.58 0)
 			(effects
 				(font
@@
 		)
 		(property "Footprint" ""
-			(at 184.15 72.39 0)
+			(at 184.15 73.66 0)
 			(effects
 				(font
@@
 		)
 		(property "Datasheet" ""
-			(at 184.15 72.39 0)
+			(at 184.15 73.66 0)
 			(effects
 				(font
@@
 		)
 		(property "Description" "Power symbol creates a global label with name \"+5V\""
-			(at 184.15 72.39 0)
+			(at 184.15 73.66 0)
 			(effects
 				(font
@@
 	(symbol
 		(lib_id "Connector:TestPoint")
-		(at 194.31 72.39 180)
+		(at 194.31 73.66 180)
 		(unit 1)
 		(exclude_from_sim no)
@@
 		(dnp no)
 		(property "Reference" "TP2"
-			(at 195.834 81.026 0)
+			(at 195.834 82.296 0)
 			(effects
 				(font
@@
 		)
 		(property "Value" "TP5V"
-			(at 196.596 78.486 0)
+			(at 196.596 79.756 0)
 			(effects
 				(font
@@
 		)
 		(property "Footprint" "TestPoint:TestPoint_Pad_D1.5mm"
-			(at 189.23 72.39 0)
+			(at 189.23 73.66 0)
 			(effects
 				(font
@@
 		)
 		(property "Datasheet" "~"
-			(at 189.23 72.39 0)
+			(at 189.23 73.66 0)
 			(effects
 				(font
@@
 		)
 		(property "Description" "test point"
-			(at 194.31 72.39 0)
+			(at 194.31 73.66 0)
 			(effects
 				(font
@@
 	(symbol
 		(lib_id "Connector:TestPoint")
-		(at 212.09 72.39 180)
+		(at 212.09 73.66 180)
 		(unit 1)
 		(exclude_from_sim no)
@@
 		(dnp no)
 		(property "Reference" "TP4"
-			(at 213.868 81.026 0)
+			(at 213.868 82.296 0)
 			(effects
 				(font
@@
 		)
 		(property "Value" "TPSW2"
-			(at 214.884 78.74 0)
+			(at 214.884 80.01 0)
 			(effects
 				(font
@@
 		)
 		(property "Footprint" "TestPoint:TestPoint_Pad_D1.5mm"
-			(at 207.01 72.39 0)
+			(at 207.01 73.66 0)
 			(effects
 				(font
@@
 		)
 		(property "Datasheet" "~"
-			(at 207.01 72.39 0)
+			(at 207.01 73.66 0)
 			(effects
 				(font
@@
 		)
 		(property "Description" "test point"
-			(at 212.09 72.39 0)
+			(at 212.09 73.66 0)
 			(effects
 				(font
@@
 	(symbol
 		(lib_id "power:+5V")
-		(at 67.31 31.75 0)
-		(unit 1)
-		(exclude_from_sim no)
-		(in_bom yes)
-		(on_board yes)
-		(dnp no)
-		(fields_autoplaced yes)
-		(property "Reference" "#PWR05"
-			(at 67.31 35.56 0)
-			(effects
-				(font
-					(size 1.27 1.27)
-				)
-				(hide yes)
-			)
-		)
-		(property "Value" "+5V"
-			(at 67.31 26.67 0)
-			(effects
-				(font
-					(size 1.27 1.27)
-				)
-			)
-		)
-		(property "Footprint" ""
-			(at 67.31 31.75 0)
-			(effects
-				(font
-					(size 1.27 1.27)
-				)
-				(hide yes)
-			)
-		)
-		(property "Datasheet" ""
-			(at 67.31 31.75 0)
-			(effects
-				(font
-					(size 1.27 1.27)
-				)
-				(hide yes)
-			)
-		)
-		(property "Description" "Power symbol creates a global label with name \"+5V\""
-			(at 67.31 31.75 0)
-			(effects
-				(font
-					(size 1.27 1.27)
-				)
-				(hide yes)
-			)
-		)
-		(pin "1"
-		)
-		(instances
-			(project "CNChess_KiCad"
-				(path "/217afebd-c7e0-4ae3-a41a-8884648524ec"
-					(reference "#PWR05")
-					(unit 1)
-				)
-			)
-		)
-	)
-	(symbol
-		(lib_id "power:+5V")
 		(at 129.54 161.29 0)
 		(unit 1)
@@
 	)
 	(symbol
-		(lib_id "power:+5V")
-		(at 194.31 72.39 0)
-		(unit 1)
-		(exclude_from_sim no)
-		(in_bom yes)
-		(on_board yes)
-		(dnp no)
-		(fields_autoplaced yes)
-		(property "Reference" "#PWR011"
-			(at 194.31 76.2 0)
-			(effects
-				(font
-					(size 1.27 1.27)
-				)
-				(hide yes)
-			)
-		)
-		(property "Value" "+5V"
-			(at 194.31 67.31 0)
-			(effects
-				(font
-					(size 1.27 1.27)
-				)
-			)
-		)
-		(property "Footprint" ""
-			(at 194.31 72.39 0)
-			(effects
-				(font
-					(size 1.27 1.27)
-				)
-				(hide yes)
-			)
-		)
-		(property "Datasheet" ""
-			(at 194.31 72.39 0)
-			(effects
-				(font
-					(size 1.27 1.27)
-				)
-				(hide yes)
-			)
-		)
-		(property "Description" "Power symbol creates a global label with name \"+5V\""
-			(at 194.31 72.39 0)
-			(effects
-				(font
-					(size 1.27 1.27)
-				)
-				(hide yes)
-			)
-		)
-		(pin "1"
-		)
-		(instances
-			(project "CNChess_KiCad"
-				(path "/217afebd-c7e0-4ae3-a41a-8884648524ec"
-					(reference "#PWR011")
-					(unit 1)
-				)
-			)
-		)
-	)
-	(symbol
 		(lib_id "power:GND")
 		(at 154.94 44.45 0)
@@
 	(symbol
 		(lib_id "Connector:TestPoint")
-		(at 184.15 72.39 180)
+		(at 184.15 73.66 180)
 		(unit 1)
 		(exclude_from_sim no)
@@
 		(dnp no)
 		(property "Reference" "TP1"
-			(at 185.674 81.026 0)
+			(at 185.674 82.296 0)
 			(effects
 				(font
@@
 		)
 		(property "Value" "TP12V"
-			(at 186.944 78.486 0)
+			(at 186.944 79.756 0)
 			(effects
 				(font
@@
 		)
 		(property "Footprint" "TestPoint:TestPoint_Pad_D1.5mm"
-			(at 179.07 72.39 0)
+			(at 179.07 73.66 0)
 			(effects
 				(font
@@
 		)
 		(property "Datasheet" "~"
-			(at 179.07 72.39 0)
+			(at 179.07 73.66 0)
 			(effects
 				(font
@@
 		)
 		(property "Description" "test point"
-			(at 184.15 72.39 0)
+			(at 184.15 73.66 0)
 			(effects
 				(font
