File: CNChess_KiCad/CNChess_KiCad.kicad_pcb (KiCad board)
At the start: 2 copper layers, 83.7 x 50.9 mm, 32 parts, among them J1 Barrel_Jack, J2 Motor1, J3 Motor2, J4 Servomotor, J5 Fan, SW1 LSW1, SW2 LSW2, SW3 OOSW, U1 ESP32C3, U2 Power_Regulator

Commit message: update elec et TBsem5
Parts:
- D3: value LED -> X
- D4: value LED -> Y
- moved C3 0.60 mm to (153.3, 86.5)
- moved C4 0.60 mm to (166.3, 86.5)
- moved C2 0.25 mm to (134.4, 114.7)
Connections:
- J4 pad 2: Net-(J4-Pin_2) -> +5V_buck
- TP2 pad 1: +5V -> +5V_buck
- U1 pad 14: +5V -> unconnected-(U1-5V-Pad14)
- U2 pad 5: Net-(J4-Pin_2) -> +5V_buck
Routing:
- net +5V: track 107.1 -> 0.00 mm
- net +5V_buck: track 0.00 -> 74.1 mm
- net +12V: track 138.4 -> 163.5 mm
- net Net-(J4-Pin_2): track 16.7 -> 0.00 mm
- net Net-(J3-Pin_1): track 74.2 -> 68.3 mm
- net Net-(J3-Pin_2): track 71.5 -> 66.0 mm
- net Net-(J2-Pin_1): track 44.8 -> 47.9 mm
- net Net-(J2-Pin_2): track 47.8 -> 50.5 mm
- net Net-(J2-Pin_3): track 50.6 -> 52.8 mm
- net Net-(J2-Pin_4): track 53.6 -> 55.3 mm
- net DIR2: track 32.5 -> 31.6 mm
- net STEP2: track 31.0 -> 30.1 mm
- net +3V3: track 130.5 -> 131.3 mm
- net Net-(J3-Pin_3): track 68.8 -> 68.1 mm
- net GND: vias 3 -> 85
Other:
- board text added: "CNChess"
- board text added: "Celeste & Julien & Christophe & Emanuel & Thomas & Zacharie"
- board text added: "Design par Julien & Celeste Genie robotique Promotion 70 Hiver 2026 Projet S4"

Commit message: pcb ready
Routing:
- net GND: vias 85 -> 66
